File: PCB/RevB/coop assistant.brd (EAGLE design)
At the start: 86.4 x 155.7 mm, 116 parts, among them IC1 74LVC1G06DBV, IC2 74LVC1G06DBV, Q1 IRFR4105, Q2 IRFR4105, Q3 IRFR4105, Q4 IRFR4105, Q5 IRFR4105, Q6 X0202MN_5BA4, T1 BC847, T2 BC847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

Commit message: Rev B PCB Update
Parts:
- added C3: 0.1u, rcl:C0805
- added D6: SS2FL4, Jeremy Custom Parts:SMF
- added R35: 100, resistor:R2512
- D5: value 15V -> 18V
Connections:
- new net +12V_MOTOR: C16.POS, C24.POS, C28.POS, D6.K, Q2.3, Q4.3
- new net MOTOR_SNUB_RC: C3.1, R35.2
- net +12V: now also D6.A; no longer C16.POS, C24.POS, C28.POS, Q2.3, Q4.3
- net AHS: now also R35.1
- net BHS: now also C3.2
Routing:
- net MOTOR_SNUB_RC: track 0.00 -> 4.19 mm
- net BHS: track 108.5 -> 111.8 mm
- net +12V_MOTOR: track 0.00 -> 2.62 mm
- net +12V: track 140.0 -> 142.3 mm
- net AHS: track 93.9 -> 96.1 mm
- added copper zone on layer 1, net +12V_MOTOR
Changed lines of the file:
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@@
 <attribute name="VALUE" x="21.209" y="118.364" size="1.27" layer="27"/>
 </element>
-<element name="D5" library="diode" library_urn="urn:adsk.eagle:library:210" package="SOT23" package3d_urn="urn:adsk.eagle:package:43389/2" value="15V" x="26.67" y="124.968" smashed="yes">
+<element name="D5" library="diode" library_urn="urn:adsk.eagle:library:210" package="SOT23" package3d_urn="urn:adsk.eagle:package:43389/2" value="18V" x="26.67" y="124.968" smashed="yes">
 <attribute name="NAME" x="25.019" y="127.127" size="1.5" layer="25"/>
 <attribute name="POPULARITY" value="3" x="26.67" y="124.968" size="1.778" layer="27" display="off"/>
@@
 <attribute name="NAME" x="36.195" y="63.246" size="1.27" layer="25" rot="R180"/>
 <attribute name="VALUE" x="36.195" y="67.056" size="1.27" layer="27" rot="R180"/>
+</element>
+<element name="D6" library="Jeremy Custom Parts" library_urn="urn:adsk.eagle:library:33094030" package="SMF" package3d_urn="urn:adsk.eagle:package:33093907/4" value="SS2FL4" x="2.54" y="34.544" smashed="yes" rot="R90">
+<attribute name="NAME" x="0.8051" y="34.544" size="1.27" layer="25" rot="R90" align="bottom-center"/>
+<attribute name="VALUE" x="-2.0751" y="34.544" size="1.27" layer="27" rot="R90" align="top-center"/>
+</element>
+<element name="R35" library="resistor" library_urn="urn:adsk.eagle:library:348" package="R2512" package3d_urn="urn:adsk.eagle:package:23545/2" value="100" x="73.406" y="10.16" smashed="yes" rot="R270">
+<attribute name="NAME" x="75.311" y="12.7" size="1.27" layer="25" rot="R270"/>
+<attribute name="VALUE" x="70.231" y="12.7" size="1.27" layer="27" rot="R270"/>
+</element>
+<element name="C3" library="rcl" library_urn="urn:adsk.eagle:library:334" package="C0805" package3d_urn="urn:adsk.eagle:package:23617/2" value="0.1u" x="69.342" y="6.096" smashed="yes" rot="R270">
+<attribute name="NAME" x="70.612" y="7.366" size="1.27" layer="25" rot="R270"/>
+<attribute name="POPULARITY" value="88" x="69.342" y="6.096" size="1.5" layer="27" ratio="11" rot="R270" display="off"/>
+<attribute name="SPICEPREFIX" value="C" x="69.342" y="6.096" size="1.5" layer="27" ratio="11" rot="R270" display="off"/>
+<attribute name="VALUE" x="66.802" y="7.366" size="1.27" layer="27" rot="R270"/>
+<attribute name="VOLTAGE" value="100V" x="69.342" y="6.096" size="1.778" layer="27" rot="R270" display="off"/>
 </element>
 </elements>
@@
 <contactref element="D2" pad="A"/>
 <contactref element="D3" pad="A"/>
-<contactref element="Q4" pad="3"/>
-<contactref element="Q2" pad="3"/>
 <contactref element="F3" pad="2"/>
 <contactref element="D4" pad="C"/>
@@
 <vertex x="10.922" y="124.206"/>
 <vertex x="3.556" y="116.84"/>
-<vertex x="3.556" y="1.016"/>
-<vertex x="1.016" y="1.016"/>
+<vertex x="3.556" y="37.592"/>
+<vertex x="1.016" y="37.592"/>
 </polygon>
 <wire x1="21.59" y1="130.588" x2="19.082" y2="130.588" width="1.27" layer="1"/>
@@
 <wire x1="40.386" y1="37.2745" x2="43.18" y2="37.2745" width="1.27" layer="1"/>
 <wire x1="43.18" y1="37.2745" x2="43.18" y2="47.498" width="1.27" layer="1"/>
-<polygon width="0.254" layer="1" thermals="no">
-<vertex x="3.363309375" y="31.496"/>
-<vertex x="13.462" y="31.496"/>
-<vertex x="13.462" y="4.064"/>
-<vertex x="3.048" y="4.064"/>
-</polygon>
 <wire x1="67.31" y1="46.482" x2="68.072" y2="47.244" width="2.54" layer="1"/>
 <wire x1="68.072" y1="47.244" x2="70.866" y2="47.244" width="2.54" layer="1"/>
@@
 <wire x1="25.4" y1="29.21" x2="26.228" y2="29.21" width="0.508" layer="1"/>
 <wire x1="26.228" y1="29.21" x2="26.366" y2="29.348" width="0.508" layer="1"/>
-<contactref element="C16" pad="POS"/>
-<contactref element="C28" pad="POS"/>
-<contactref element="C24" pad="POS"/>
+<contactref element="D6" pad="A"/>
+<wire x1="2.54" y1="35.844" x2="2.54" y2="38.1" width="1.27" layer="1"/>
 </signal>
 <signal name="A_ISENSE" class="4">
@@
 <wire x1="28.742" y1="21.844" x2="28.742" y2="17.74" width="1.27" layer="1"/>
 <wire x1="28.742" y1="17.74" x2="33.02" y2="13.462" width="1.27" layer="1"/>
-<wire x1="71.2001" y1="5.08" x2="81.2796" y2="15.1595" width="1.27" layer="1"/>
-<wire x1="34.544" y1="5.08" x2="71.2001" y2="5.08" width="1.27" layer="1"/>
+<wire x1="70.8656" y1="15.1595" x2="73.406" y2="15.1595" width="1.27" layer="1"/>
+<wire x1="73.406" y1="15.1595" x2="81.2796" y2="15.1595" width="1.27" layer="1"/>
+<wire x1="70.8656" y1="15.1595" x2="60.7861" y2="5.08" width="1.27" layer="1"/>
+<wire x1="34.544" y1="5.08" x2="60.7861" y2="5.08" width="1.27" layer="1"/>
+<contactref element="R35" pad="1"/>
+<wire x1="73.406" y1="12.96" x2="73.406" y2="15.1595" width="1.27" layer="1"/>
 </signal>
 <signal name="BHS" class="5">
@@
 <wire x1="24.892" y1="17.78" x2="26.162" y2="16.51" width="0.4064" layer="1"/>
 <wire x1="26.67" y1="14.478" x2="26.71" y2="14.478" width="0.4064" layer="1"/>
-<wire x1="73.9941" y1="2.794" x2="81.2796" y2="10.0795" width="1.27" layer="1"/>
-<wire x1="30.226" y1="2.794" x2="73.9941" y2="2.794" width="1.27" layer="1"/>
+<wire x1="81.2796" y1="8.5555" x2="75.5181" y2="2.794" width="1.27" layer="1"/>
+<wire x1="81.2796" y1="8.5555" x2="81.2796" y2="10.0795" width="1.27" layer="1"/>
+<wire x1="30.226" y1="2.794" x2="69.342" y2="2.794" width="1.27" layer="1"/>
+<contactref element="C3" pad="2"/>
+<wire x1="69.342" y1="2.794" x2="75.5181" y2="2.794" width="1.27" layer="1"/>
+<wire x1="69.342" y1="5.146" x2="69.342" y2="2.794" width="1.27" layer="1"/>
 </signal>
 <signal name="AHO" class="3">
@@
 <wire x1="66.04" y1="134.0634" x2="65.9914" y2="134.112" width="0.3048" layer="1"/>
 </signal>
+<signal name="+12V_MOTOR" class="1">
+<contactref element="C16" pad="POS"/>
+<contactref element="C28" pad="POS"/>
+<contactref element="C24" pad="POS"/>
+<contactref element="D6" pad="K"/>
+<contactref element="Q4" pad="3"/>
+<contactref element="Q2" pad="3"/>
+<polygon width="0.1524" layer="1" thermals="no">
+<vertex x="1.524" y="31.496"/>
+<vertex x="11.938" y="31.496"/>
+<vertex x="13.97" y="29.464"/>
+<vertex x="13.97" y="6.604"/>
+<vertex x="1.524" y="6.604"/>
+</polygon>
+<wire x1="2.54" y1="33.244" x2="2.54" y2="30.988" width="1.27" layer="1"/>
+<wire x1="2.54" y1="30.988" x2="2.794" y2="30.734" width="1.27" layer="1"/>
+</signal>
+<signal name="MOTOR_SNUB_RC" class="1">
+<contactref element="R35" pad="2"/>
+<contactref element="C3" pad="1"/>
+<wire x1="69.342" y1="7.046" x2="70.8" y2="7.046" width="1.27" layer="1"/>
+<wire x1="71.114" y1="7.36" x2="73.406" y2="7.36" width="1.27" layer="1"/>
+<wire x1="70.8" y1="7.046" x2="71.114" y2="7.36" width="1.27" layer="1"/>
+</signal>
 </signals>
