File: PCB/RevB/coop assistant.sch (EAGLE design)
At the start: 116 parts, among them IC1 74LVC1G06DBV, IC2 74LVC1G06DBV, Q1 IRFR4105, Q2 IRFR4105, Q3 IRFR4105, Q4 IRFR4105, Q5 IRFR4105, Q6 X0202MN_5BA4, T1 BC847, T2 BC847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

Commit message: Rev B PCB Update
Parts:
- added C3: 0.1u, rcl:C-EUC0805
- added D6: SS2FL4, Jeremy Custom Parts:SS2FL4
- added R35: 100, resistor:R-US_R2512
- D5: value 15V -> 18V
Connections:
- new net +12V_MOTOR: C16.+, C24.+, C28.+, D6.C, Q2.D, Q4.D
- new net MOTOR_SNUB_RC: C3.1, R35.2
- net +12V: now also D6.A; no longer C16.+, C24.+, C28.+, Q2.D, Q4.D
- net AHS: now also R35.1
- net BHS: now also C3.2
Other:
- note added: "CONNECT MOTOR HERE"
- moved on the sheet: C16, C18, C19, C24, C28, Q2, Q3, Q4, Q5, R25, R26, R27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
